File: untitled.sch (EAGLE design)
At the start: 0 parts

Commit message: hello world
Parts:
- added C1, C10, C11, C12, C13, C14, C15, C16, C17, C18, C19, C2, C20, C21, C22, C23, C24, C25, C26, C27, C28, C29, C3, C30, C31, C32, C33, C34, C35, C36, C37, C38, C39, C4, C40, C41, C42, C43, C44, C5, C6, C7, C8, C9: (no value), resistor:C-EU025-024X044
Connections:
- new net N$1: C17.1, C4.2
- new net N$2: C35.1, C36.2
Changed lines of the file:
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@@
 <grid distance="0.1" unitdist="inch" unit="inch" style="lines" multiple="1" display="no" altdistance="0.01" altunitdist="inch" altunit="inch"/>
 <layers>
+<layer number="1" name="Top" color="4" fill="1" visible="no" active="no"/>
+<layer number="16" name="Bottom" color="1" fill="1" visible="no" active="no"/>
+<layer number="17" name="Pads" color="2" fill="1" visible="no" active="no"/>
+<layer number="18" name="Vias" color="2" fill="1" visible="no" active="no"/>
+<layer number="19" name="Unrouted" color="6" fill="1" visible="no" active="no"/>
+<layer number="20" name="Dimension" color="15" fill="1" visible="no" active="no"/>
+<layer number="21" name="tPlace" color="7" fill="1" visible="no" active="no"/>
+<layer number="22" name="bPlace" color="7" fill="1" visible="no" active="no"/>
+<layer number="23" name="tOrigins" color="15" fill="1" visible="no" active="no"/>
+<layer number="24" name="bOrigins" color="15" fill="1" visible="no" active="no"/>
+<layer number="25" name="tNames" color="7" fill="1" visible="no" active="no"/>
+<layer number="26" name="bNames" color="7" fill="1" visible="no" active="no"/>
+<layer number="27" name="tValues" color="7" fill="1" visible="no" active="no"/>
+<layer number="28" name="bValues" color="7" fill="1" visible="no" active="no"/>
+<layer number="29" name="tStop" color="7" fill="3" visible="no" active="no"/>
+<layer number="30" name="bStop" color="7" fill="6" visible="no" active="no"/>
+<layer number="31" name="tCream" color="7" fill="4" visible="no" active="no"/>
+<layer number="32" name="bCream" color="7" fill="5" visible="no" active="no"/>
+<layer number="33" name="tFinish" color="6" fill="3" visible="no" active="no"/>
+<layer number="34" name="bFinish" color="6" fill="6" visible="no" active="no"/>
+<layer number="35" name="tGlue" color="7" fill="4" visible="no" active="no"/>
+<layer number="36" name="bGlue" color="7" fill="5" visible="no" active="no"/>
+<layer number="37" name="tTest" color="7" fill="1" visible="no" active="no"/>
+<layer number="38" name="bTest" color="7" fill="1" visible="no" active="no"/>
+<layer number="39" name="tKeepout" color="4" fill="11" visible="no" active="no"/>
+<layer number="40" name="bKeepout" color="1" fill="11" visible="no" active="no"/>
+<layer number="41" name="tRestrict" color="4" fill="10" visible="no" active="no"/>
+<layer number="42" name="bRestrict" color="1" fill="10" visible="no" active="no"/>
+<layer number="43" name="vRestrict" color="2" fill="10" visible="no" active="no"/>
+<layer number="44" name="Drills" color="7" fill="1" visible="no" active="no"/>
+<layer number="45" name="Holes" color="7" fill="1" visible="no" active="no"/>
+<layer number="46" name="Milling" color="3" fill="1" visible="no" active="no"/>
+<layer number="47" name="Measures" color="7" fill="1" visible="no" active="no"/>
+<layer number="48" name="Document" color="7" fill="1" visible="no" active="no"/>
+<layer number="49" name="Reference" color="7" fill="1" visible="no" active="no"/>
+<layer number="51" name="tDocu" color="7" fill="1" visible="no" active="no"/>
+<layer number="52" name="bDocu" color="7" fill="1" visible="no" active="no"/>
 <layer number="91" name="Nets" color="2" fill="1" visible="yes" active="yes"/>
 <layer number="92" name="Busses" color="1" fill="1" visible="yes" active="yes"/>
@@
 </classes>
 <parts>
+<part name="C1" library="resistor" deviceset="C-EU" device="025-024X044"/>
+<part name="C2" library="resistor" deviceset="C-EU" device="025-024X044"/>
+<part name="C3" library="resistor" deviceset="C-EU" device="025-024X044"/>
+<part name="C4" library="resistor" deviceset="C-EU" device="025-024X044"/>
+<part name="C5" library="resistor" deviceset="C-EU" device="025-024X044"/>
+<part name="C6" library="resistor" deviceset="C-EU" device="025-024X044"/>
+<part name="C7" library="resistor" deviceset="C-EU" device="025-024X044"/>
+<part name="C8" library="resistor" deviceset="C-EU" device="025-024X044"/>
+<part name="C9" library="resistor" deviceset="C-EU" device="025-024X044"/>
+<part name="C10" library="resistor" deviceset="C-EU" device="025-024X044"/>
+<part name="C11" library="resistor" deviceset="C-EU" device="025-024X044"/>
+<part name="C12" library="resistor" deviceset="C-EU" device="025-024X044"/>
+<part name="C13" library="resistor" deviceset="C-EU" device="025-024X044"/>
+<part name="C14" library="resistor" deviceset="C-EU" device="025-024X044"/>
+<part name="C15" library="resistor" deviceset="C-EU" device="025-024X044"/>
+<part name="C16" library="resistor" deviceset="C-EU" device="025-024X044"/>
+<part name="C17" library="resistor" deviceset="C-EU" device="025-024X044"/>
+<part name="C18" library="resistor" deviceset="C-EU" device="025-024X044"/>
+<part name="C19" library="resistor" deviceset="C-EU" device="025-024X044"/>
+<part name="C20" library="resistor" deviceset="C-EU" device="025-024X044"/>
+<part name="C21" library="resistor" deviceset="C-EU" device="025-024X044"/>
+<part name="C22" library="resistor" deviceset="C-EU" device="025-024X044"/>
+<part name="C23" library="resistor" deviceset="C-EU" device="025-024X044"/>
+<part name="C24" library="resistor" deviceset="C-EU" device="025-024X044"/>
+<part name="C25" library="resistor" deviceset="C-EU" device="025-024X044"/>
+<part name="C26" library="resistor" deviceset="C-EU" device="025-024X044"/>
+<part name="C27" library="resistor" deviceset="C-EU" device="025-024X044"/>
+<part name="C28" library="resistor" deviceset="C-EU" device="025-024X044"/>
+<part name="C29" library="resistor" deviceset="C-EU" device="025-024X044"/>
+<part name="C30" library="resistor" deviceset="C-EU" device="025-024X044"/>
+<part name="C31" library="resistor" deviceset="C-EU" device="025-024X044"/>
+<part name="C32" library="resistor" deviceset="C-EU" device="025-024X044"/>
+<part name="C33" library="resistor" deviceset="C-EU" device="025-024X044"/>
+<part name="C34" library="resistor" deviceset="C-EU" device="025-024X044"/>
+<part name="C35" library="resistor" deviceset="C-EU" device="025-024X044"/>
+<part name="C36" library="resistor" deviceset="C-EU" device="025-024X044"/>
+<part name="C37" library="resistor" deviceset="C-EU" device="025-024X044"/>
+<part name="C38" library="resistor" deviceset="C-EU" device="025-024X044"/>
+<part name="C39" library="resistor" deviceset="C-EU" device="025-024X044"/>
+<part name="C40" library="resistor" deviceset="C-EU" device="025-024X044"/>
+<part name="C41" library="resistor" deviceset="C-EU" device="025-024X044"/>
+<part name="C42" library="resistor" deviceset="C-EU" device="025-024X044"/>
+<part name="C43" library="resistor" deviceset="C-EU" device="025-024X044"/>
+<part name="C44" library="resistor" deviceset="C-EU" device="025-024X044"/>
 </parts>
 <sheets>
@@
 </plain>
 <instances>
+<instance part="C1" gate="G$1" x="35.56" y="78.74"/>
+<instance part="C2" gate="G$1" x="48.26" y="58.42"/>
+<instance part="C3" gate="G$1" x="114.3" y="63.5"/>
+<instance part="C4" gate="G$1" x="99.06" y="88.9"/>
+<instance part="C5" gate="G$1" x="71.12" y="38.1"/>
+<instance part="C6" gate="G$1" x="76.2" y="17.78"/>
+<instance part="C7" gate="G$1" x="-15.24" y="43.18"/>
+<instance part="C8" gate="G$1" x="88.9" y="43.18"/>
+<instance part="C9" gate="G$1" x="88.9" y="17.78"/>
+<instance part="C10" gate="G$1" x="20.32" y="35.56"/>
+<instance part="C11" gate="G$1" x="55.88" y="78.74"/>
+<instance part="C12" gate="G$1" x="83.82" y="60.96"/>
+<instance part="C13" gate="G$1" x="66.04" y="33.02"/>
+<instance part="C14" gate="G$1" x="53.34" y="15.24"/>
+<instance part="C15" gate="G$1" x="93.98" y="15.24"/>
+<instance part="C16" gate="G$1" x="137.16" y="48.26"/>
+<instance part="C17" gate="G$1" x="99.06" y="81.28"/>
+<instance part="C18" gate="G$1" x="35.56" y="81.28"/>
+<instance part="C19" gate="G$1" x="48.26" y="27.94"/>
+<instance part="C20" gate="G$1" x="66.04" y="12.7"/>
+<instance part="C21" gate="G$1" x="17.78" y="58.42"/>
+<instance part="C22" gate="G$1" x="25.4" y="81.28"/>
+<instance part="C23" gate="G$1" x="2.54" y="38.1"/>
+<instance part="C24" gate="G$1" x="58.42" y="-2.54"/>
+<instance part="C25" gate="G$1" x="17.78" y="-7.62"/>
+<instance part="C26" gate="G$1" x="20.32" y="2.54"/>
+<instance part="C27" gate="G$1" x="43.18" y="40.64"/>
+<instance part="C28" gate="G$1" x="45.72" y="45.72"/>
+<instance part="C29" gate="G$1" x="27.94" y="27.94"/>
+<instance part="C30" gate="G$1" x="35.56" y="-2.54"/>
+<instance part="C31" gate="G$1" x="55.88" y="-20.32"/>
+<instance part="C32" gate="G$1" x="81.28" y="2.54"/>
+<instance part="C33" gate="G$1" x="99.06" y="-10.16"/>
+<instance part="C34" gate="G$1" x="111.76" y="5.08"/>
+<instance part="C35" gate="G$1" x="106.68" y="15.24"/>
+<instance part="C36" gate="G$1" x="106.68" y="22.86"/>
+<instance part="C37" gate="G$1" x="93.98" y="27.94"/>
+<instance part="C38" gate="G$1" x="86.36" y="40.64"/>
+<instance part="C39" gate="G$1" x="81.28" y="60.96"/>
+<instance part="C40" gate="G$1" x="73.66" y="73.66"/>
+<instance part="C41" gate="G$1" x="83.82" y="83.82"/>
+<instance part="C42" gate="G$1" x="111.76" y="86.36"/>
+<instance part="C43" gate="G$1" x="121.92" y="76.2"/>
+<instance part="C44" gate="G$1" x="121.92" y="45.72"/>
 </instances>
 <busses>
 </busses>
 <nets>
+<net name="N$1" class="0">
+<segment>
+<pinref part="C4" gate="G$1" pin="2"/>
+<pinref part="C17" gate="G$1" pin="1"/>
+</segment>
+</net>
+<net name="N$2" class="0">
+<segment>
+<pinref part="C35" gate="G$1" pin="1"/>
+<pinref part="C36" gate="G$1" pin="2"/>
+</segment>
+</net>
 </nets>
 </sheet>
